Commit message: up

File: zbot_stella_n2_description/urdf/zbot_stella_n2.urdf.xacro (robot description, xacro)
@@ -64,4 +64,10 @@
   </xacro:macro>
   <link name="base_link"></link>
+  <link name="base_footprint"></link>
+  <joint name="base_footprint_joint" type="fixed">
+    <origin xyz="0 0 ${-1 *(footprint_vertical_offset + chassis_height/2)}" rpy="0 0 0"/>
+    <parent link="base_link"/>
+    <child link="base_footprint"/>
+  </joint>
   <joint name="chassis_joint" type="fixed">
     <origin xyz="0 0 0" rpy="0 0 0"/>

Commit message: up

File: zbot_stella_n2_description/urdf/zbot_stella_n2.urdf.xacro (robot description, xacro)
@@ -129,4 +129,10 @@
     <child link="ball_caster_link"/>
   </joint>
+  <link name="imu_link"></link>
+  <joint name="imu_joint" type="fixed">
+    <origin xyz="${0.025-chassis_length/2} 0 ${chassis_height/2}" rpy="0 0 0"/>
+    <parent link="chassis_link"/>
+    <child link="imu_link"/>
+  </joint>
   <!-- ROS2 controls -->
   <ros2_control name="zbot_stella_n2_hardware" type="system">

Commit message: up

File: zbot_stella_n2_description/urdf/zbot_stella_n2.urdf.xacro (robot description, xacro)
@@ -67,6 +67,6 @@
   <joint name="base_footprint_joint" type="fixed">
     <origin xyz="0 0 ${-1 *(footprint_vertical_offset + chassis_height/2)}" rpy="0 0 0"/>
-    <parent link="base_link"/>
-    <child link="base_footprint"/>
+    <parent link="base_footprint"/>
+    <child link="base_link"/>
   </joint>
   <joint name="chassis_joint" type="fixed">

Commit message: up

File: zbot_stella_n2_description/urdf/zbot_stella_n2.urdf.xacro (robot description, xacro)
@@ -129,4 +129,5 @@
     <child link="ball_caster_link"/>
   </joint>
+  <!-- accessories -->
   <link name="imu_link"></link>
   <joint name="imu_joint" type="fixed">
@@ -134,4 +135,10 @@
     <parent link="chassis_link"/>
     <child link="imu_link"/>
+  </joint>
+  <link name="laser_link"></link>
+  <joint name="laser_joint" type="fixed">
+    <origin xyz="${4.5} 0 ${13.5}" rpy="0 0 0"/>
+    <parent link="chassis_link"/>
+    <child link="laser_link"/>
   </joint>
   <!-- ROS2 controls -->

Commit message: up

File: zbot_stella_n2_description/urdf/zbot_stella_n2.urdf.xacro (robot description, xacro)
@@ -138,5 +138,5 @@
   <link name="laser_link"></link>
   <joint name="laser_joint" type="fixed">
-    <origin xyz="${4.5} 0 ${13.5}" rpy="0 0 0"/>
+    <origin xyz="${0.045} 0 ${0.135}" rpy="0 0 0"/>
     <parent link="chassis_link"/>
     <child link="laser_link"/>

Commit message: up

File: zbot_stella_n2_description/urdf/zbot_stella_n2.urdf.xacro (robot description, xacro)
@@ -3,5 +3,5 @@
   <!-- https://en.wikipedia.org/wiki/List_of_moments_of_inertia#List_of_3D_inertia_tensors -->
   <xacro:arg name="is_sim" default="false"/>
-  <xacro:arg name="gazebo_controllers" default="$(find zbot_stella_n2_control)/config/control.yaml" />
+  <xacro:arg name="gazebo_controllers" default="$(find zbot_stella_n2_control)/config/gazebo_control.yaml" />
   <xacro:property name="PI" value="3.1415926535897931"/>
   <xacro:property name="footprint_vertical_offset" value="0.0085" />
@@ -53,5 +53,5 @@
       <axis xyz="0 1 0"/>
     </joint>
-    <transmission name="${prefix}_wheel_trans">
+    <!-- <transmission name="${prefix}_wheel_trans">
       <type>transmission_interface/SimpleTransmission</type>
       <joint name="${prefix}_wheel">
@@ -61,5 +61,5 @@
         <mechanicalReduction>1</mechanicalReduction>
       </actuator>
-    </transmission>
+    </transmission> -->
   </xacro:macro>
   <link name="base_link"></link>
@@ -151,5 +151,26 @@
   </ros2_control>
   <!-- Bring in simulation data for Gazebo. -->
-  <!-- <xacro:include filename="$(find zbot_stella_n2_description)/urdf/zbot_stella_n2.gazebo" /> -->
-  <xacro:include filename="$(find zbot_stella_n2_description)/urdf/accessories.urdf.xacro" />
+  <xacro:if value="$(arg is_sim)">
+    <xacro:include filename="$(find zbot_stella_n2_description)/urdf/zbot_stella_n2.gazebo" />
+  </xacro:if>
+  <xacro:unless value="$(arg is_sim)">
+    <xacro:include filename="$(find zbot_stella_n2_description)/urdf/accessories.urdf.xacro" />
+  </xacro:unless>
 </robot>
+  <!-- <ros2_control name="GazeboSystem" type="system">
+      <hardware>
+          <plugin>gazebo_ros2_control/GazeboSystem</plugin>
+      </hardware>
+      <joint name="left_wheel_joint">
+          <command_interface name="velocity">
+          </command_interface>
+          <state_interface name="position" />
+          <state_interface name="velocity" />
+      </joint>
+      <joint name="right_wheel_joint">
+          <command_interface name="velocity">
+          </command_interface>
+          <state_interface name="velocity" />
+          <state_interface name="position" />
+      </joint>
+  </ros2_control> -->
