Commit message: up

File: zbot_stella_n2_description/urdf/accessories.urdf.xacro (robot description, xacro)
@@ -1,3 +1,16 @@
 <?xml version="1.0" ?>
 <robot xmlns:xacro="http://ros.org/wiki/xacro">
+  <!-- accessories -->
+  <link name="imu_link"></link>
+  <joint name="imu_joint" type="fixed">
+    <origin xyz="${0.025-chassis_length/2} 0 ${chassis_height/2}" rpy="0 0 0"/>
+    <parent link="chassis_link"/>
+    <child link="imu_link"/>
+  </joint>
+  <link name="laser_link"></link>
+  <joint name="laser_joint" type="fixed">
+    <origin xyz="${0.045} 0 ${0.135}" rpy="0 0 0"/>
+    <parent link="chassis_link"/>
+    <child link="laser_link"/>
+  </joint>
 </robot>

File: zbot_stella_n2_description/urdf/zbot_stella_n2.urdf.xacro (robot description, xacro)
@@ -129,17 +129,4 @@
     <child link="ball_caster_link"/>
   </joint>
-  <!-- accessories -->
-  <link name="imu_link"></link>
-  <joint name="imu_joint" type="fixed">
-    <origin xyz="${0.025-chassis_length/2} 0 ${chassis_height/2}" rpy="0 0 0"/>
-    <parent link="chassis_link"/>
-    <child link="imu_link"/>
-  </joint>
-  <link name="laser_link"></link>
-  <joint name="laser_joint" type="fixed">
-    <origin xyz="${0.045} 0 ${0.135}" rpy="0 0 0"/>
-    <parent link="chassis_link"/>
-    <child link="laser_link"/>
-  </joint>
   <!-- ROS2 controls -->
   <ros2_control name="zbot_stella_n2_hardware" type="system">
@@ -165,3 +152,4 @@
   <!-- Bring in simulation data for Gazebo. -->
   <!-- <xacro:include filename="$(find zbot_stella_n2_description)/urdf/zbot_stella_n2.gazebo" /> -->
+  <xacro:include filename="$(find zbot_stella_n2_description)/urdf/zbot_stella_n2.urdf.xacro" />
 </robot>

Commit message: up

File: zbot_stella_n2_description/urdf/accessories.urdf.xacro (robot description, xacro)
@@ -2,11 +2,72 @@
 <robot xmlns:xacro="http://ros.org/wiki/xacro">
   <!-- accessories -->
-  <link name="imu_link"></link>
+  <link name="imu_link">
+    <visual>
+      <geometry>
+          <box size="0.036 0.039 0.005"/>
+      </geometry>
+      <material name="yellow"/>
+    </visual>
+  </link>
   <joint name="imu_joint" type="fixed">
-    <origin xyz="${0.025-chassis_length/2} 0 ${chassis_height/2}" rpy="0 0 0"/>
     <parent link="chassis_link"/>
     <child link="imu_link"/>
+    <origin xyz="${0.025-chassis_length/2} 0 ${chassis_height/2 + 0.01}" rpy="0 0 0"/>
   </joint>
-  <link name="laser_link"></link>
+  <!-- depth camera -->
+  <link name="camera_link">
+      <visual>
+          <geometry>
+              <box size="0.02 0.095 0.02"/>
+          </geometry>
+          <material name="white"/>
+      </visual>
+  </link>
+  <joint name="camera_joint" type="fixed">
+      <parent link="chassis_link"/>
+      <child link="camera_link"/>
+      <origin xyz="0.07 0 0.065" rpy="0 0 0"/>
+  </joint>
+  <link name="camera_optical_link"></link>
+  <joint name="camera_optical_joint" type="fixed">
+      <parent link="camera_link"/>
+      <child link="camera_optical_link"/>
+      <origin xyz="0 0 0" rpy="${-pi/2} 0 ${-pi/2}"/>
+  </joint>
+  <!-- realsense -->
+  <!-- <link name="realsense_link">
+    <visual name="realsense_link_visual">
+        <pose>0 0 0 -1.57 0 -1.57</pose>
+        <geometry>
+          <mesh>
+            <uri>model://zbot_stella_n2_description/models/realsense_camera/meshes/d435.dae</uri>
+          </mesh>
+        </geometry>
+    </visual>
+  </link> -->
+  <!-- lidar -->
+  <link name="laser_link">
+    <visual>
+      <geometry>
+        <cylinder radius="0.05" length="0.04"/>
+      </geometry>
+      <material name="red"/>
+    </visual>
+    <visual>
+      <origin xyz="0 0 -0.05"/>
+      <geometry>
+          <cylinder radius="0.01" length="0.1"/>
+      </geometry>
+      <material name="black"/>
+    </visual>
+    <collision>
+      <geometry>
+        <cylinder radius="0.05" length="0.04"/>
+      </geometry>
+    </collision>
+    <xacro:inertial_cylinder mass="0.1" length="0.04" radius="0.05">
+        <origin xyz="0 0 0" rpy="0 0 0"/>
+    </xacro:inertial_cylinder>
+  </link>
   <joint name="laser_joint" type="fixed">
     <origin xyz="${0.045} 0 ${0.135}" rpy="0 0 0"/>

File: zbot_stella_n2_description/urdf/zbot_stella_n2.urdf.xacro (robot description, xacro)
@@ -2,4 +2,5 @@
 <robot name="zbot_stella_n2" xmlns:xacro="http://ros.org/wiki/xacro">
   <!-- https://en.wikipedia.org/wiki/List_of_moments_of_inertia#List_of_3D_inertia_tensors -->
+  <xacro:include filename="inertial_macros.xacro"/>
   <xacro:arg name="is_sim" default="false"/>
   <xacro:arg name="gazebo_controllers" default="$(find zbot_stella_n2_control)/config/gazebo_control.yaml" />
@@ -30,5 +31,5 @@
           <cylinder radius="${wheel_radius}" length="${wheel_width}"/>
         </geometry>
-        <material name="blue"/>
+        <material name="red"/>
       </visual>
       <collision>
@@ -130,47 +131,8 @@
   </joint>
   <!-- ROS2 controls -->
-  <ros2_control name="zbot_stella_n2_hardware" type="system">
-    <hardware>
-      <xacro:if value="$(arg is_sim)">
-        <plugin>gazebo_ros2_control/GazeboSystem</plugin>
-      </xacro:if>
-      <xacro:unless value="$(arg is_sim)">
-        <!-- later -->
-      </xacro:unless>
-    </hardware>
-    <joint name="left_wheel_joint">
-      <command_interface name="velocity"/>
-      <state_interface name="position"/>
-      <state_interface name="velocity"/>
-    </joint>
-    <joint name="right_wheel_joint">
-      <command_interface name="velocity"/>
-      <state_interface name="position"/>
-      <state_interface name="velocity"/>
-    </joint>
-  </ros2_control>
-  <!-- Bring in simulation data for Gazebo. -->
+  <xacro:include filename="$(find zbot_stella_n2_description)/urdf/ros2_control.urdf.xacro" />
   <xacro:if value="$(arg is_sim)">
     <xacro:include filename="$(find zbot_stella_n2_description)/urdf/zbot_stella_n2.gazebo" />
   </xacro:if>
-  <xacro:unless value="$(arg is_sim)">
-    <xacro:include filename="$(find zbot_stella_n2_description)/urdf/accessories.urdf.xacro" />
-  </xacro:unless>
+  <xacro:include filename="$(find zbot_stella_n2_description)/urdf/accessories.urdf.xacro" />
 </robot>
-  <!-- <ros2_control name="GazeboSystem" type="system">
-      <hardware>
-          <plugin>gazebo_ros2_control/GazeboSystem</plugin>
-      </hardware>
-      <joint name="left_wheel_joint">
-          <command_interface name="velocity">
-          </command_interface>
-          <state_interface name="position" />
-          <state_interface name="velocity" />
-      </joint>
-      <joint name="right_wheel_joint">
-          <command_interface name="velocity">
-          </command_interface>
-          <state_interface name="velocity" />
-          <state_interface name="position" />
-      </joint>
-  </ros2_control> -->

Commit message: up

File: zbot_stella_n2_description/urdf/accessories.urdf.xacro (robot description, xacro)
@@ -13,5 +13,5 @@
     <parent link="chassis_link"/>
     <child link="imu_link"/>
-    <origin xyz="${0.025-chassis_length/2} 0 ${chassis_height/2 + 0.01}" rpy="0 0 0"/>
+    <origin xyz="${0.025-chassis_length/2} 0 ${chassis_height/2 + 0.015}" rpy="0 0 0"/>
   </joint>
   <!-- depth camera -->
@@ -27,12 +27,18 @@
       <parent link="chassis_link"/>
       <child link="camera_link"/>
-      <origin xyz="0.07 0 0.065" rpy="0 0 0"/>
+      <origin xyz="0.07 0 0.105" rpy="0 0 0"/>
   </joint>
-  <link name="camera_optical_link"></link>
+  <link name="front_rscam_link"></link>
+  <joint name="front_rscam_joint" type="fixed">
+      <parent link="camera_link"/>
+      <child link="front_rscam_link"/>
+      <origin xyz="0 0 0" rpy="0 0 0"/>
+  </joint>
+  <!-- <link name="camera_optical_link"></link>
   <joint name="camera_optical_joint" type="fixed">
       <parent link="camera_link"/>
       <child link="camera_optical_link"/>
       <origin xyz="0 0 0" rpy="${-pi/2} 0 ${-pi/2}"/>
-  </joint>
+  </joint> -->
   <!-- realsense -->
   <!-- <link name="realsense_link">
@@ -55,7 +61,7 @@
     </visual>
     <visual>
-      <origin xyz="0 0 -0.05"/>
+      <origin xyz="0 0 -0.1"/>
       <geometry>
-          <cylinder radius="0.01" length="0.1"/>
+          <cylinder radius="0.01" length="0.2"/>
       </geometry>
       <material name="black"/>
@@ -71,7 +77,21 @@
   </link>
   <joint name="laser_joint" type="fixed">
-    <origin xyz="${0.045} 0 ${0.135}" rpy="0 0 0"/>
+    <origin xyz="${0.045} 0 ${0.185}" rpy="0 0 0"/>
     <parent link="chassis_link"/>
     <child link="laser_link"/>
   </joint>
+  <!-- gnss -->
+  <link name="gnss_link">
+    <visual>
+      <geometry>
+          <box size="0.036 0.039 0.005"/>
+      </geometry>
+      <material name="red"/>
+    </visual>
+  </link>
+  <joint name="gnss_joint" type="fixed">
+    <parent link="chassis_link"/>
+    <child link="gnss_link"/>
+    <origin xyz="${0.025-chassis_length/2} 0 ${chassis_height/2 + 0.095}" rpy="0 0 0"/>
+  </joint>
 </robot>

Commit message: Add UWB tag link and joint to URDF; update EKF configuration comments for clarity

File: zbot_stella_n2_description/urdf/accessories.urdf.xacro (robot description, xacro)
@@ -95,3 +95,11 @@
     <origin xyz="${0.025-chassis_length/2} 0 ${chassis_height/2 + 0.095}" rpy="0 0 0"/>
   </joint>
+  <!-- uwb tag -->
+  <link name="uwb_tag_link">
+  </link>
+  <joint name="uwb_tag_joint" type="fixed">
+    <parent link="chassis_link"/>
+    <child link="uwb_tag_link"/>
+    <origin xyz="${0.025-chassis_length/2} 0 ${chassis_height/2 + 0.015 + 0.22}" rpy="0 0 0"/>
+  </joint>
 </robot>
